Commit message: Tried removing light

File: husarion_ugv_description/urdf/common/gazebo.urdf.xacro (robot description, xacro)
@@ -99,5 +99,5 @@
   </xacro:macro>
   <!-- Lights -->
-  <xacro:macro name="light" params="reference_frame name topic namespace:=''">
+  <!-- <xacro:macro name="light" params="reference_frame name topic namespace:=''">
     <gazebo>
       <plugin filename="LEDStrip" name="husarion_ugv_gazebo::LEDStrip">
@@ -131,4 +131,4 @@
       </light>
     </gazebo>
-  </xacro:macro>
+  </xacro:macro> -->
 </robot>

File: husarion_ugv_description/urdf/lynx/lynx_macro.urdf.xacro (robot description, xacro)
@@ -52,5 +52,5 @@
         <xacro:if value="${use_sim}">
           <plugin>husarion_ugv_gazebo/EStopSystem</plugin>
-          <param name="e_stop_initial_state">true</param>
+          <param name="e_stop_initial_state">false</param>
         </xacro:if>
         <xacro:unless value="${use_sim}">

File: husarion_ugv_description/urdf/panther/panther_macro.urdf.xacro (robot description, xacro)
@@ -52,5 +52,5 @@
         <xacro:if value="${use_sim}">
           <plugin>husarion_ugv_gazebo/EStopSystem</plugin>
-          <param name="e_stop_initial_state">true</param>
+          <param name="e_stop_initial_state">false</param>
         </xacro:if>
         <xacro:unless value="${use_sim}">
@@ -161,6 +161,6 @@
       <xacro:gazebo.controller config_file="${controller_config_file}" namespace="${namespace}" />
       <xacro:gazebo.imu reference_frame="imu_link" namespace="${namespace}" />
-      <xacro:gazebo.light reference_frame="lights_channel_1_link" name="lights_channel_1" topic="lights/channel_1_frame" namespace="${namespace}" />
-      <xacro:gazebo.light reference_frame="lights_channel_2_link" name="lights_channel_2" topic="lights/channel_2_frame" namespace="${namespace}" />
+      <!-- <xacro:gazebo.light reference_frame="lights_channel_1_link" name="lights_channel_1" topic="lights/channel_1_frame" namespace="${namespace}" />
+      <xacro:gazebo.light reference_frame="lights_channel_2_link" name="lights_channel_2" topic="lights/channel_2_frame" namespace="${namespace}" /> -->
     </xacro:if>
   </xacro:macro>

Commit message: rm estartplugin and added gz_ros2_control

File: husarion_ugv_description/urdf/common/gazebo.urdf.xacro (robot description, xacro)
@@ -30,5 +30,5 @@
   <xacro:macro name="controller" params="config_file namespace:=''">
     <gazebo>
-      <plugin filename="gz_ros2_control-system" name="gz_ros2_control::GazeboSimROS2ControlPlugin">
+      <plugin filename="libgz_ros2_control-system.so" name="gz_ros2_control::GazeboSimROS2ControlPlugin">
         <parameters>${config_file}</parameters>
         <ros>
@@ -98,37 +98,3 @@
     </gazebo>
   </xacro:macro>
-  <!-- Lights -->
-  <!-- <xacro:macro name="light" params="reference_frame name topic namespace:=''">
-    <gazebo>
-      <plugin filename="LEDStrip" name="husarion_ugv_gazebo::LEDStrip">
-        <light_name>${name}</light_name>
-        <topic>${topic}</topic>
-        <namespace>${namespace}</namespace>
-        <frequency>10</frequency>
-        <width>0.5</width>
-        <height>0.015</height>
-      </plugin>
-    </gazebo>
-    <gazebo reference="${reference_frame}">
-      <light name="${name}" type="spot">
-        <cast_shadows>true</cast_shadows>
-        <visualize>0</visualize>
-        <diffuse>1.0 1.0 1.0</diffuse>
-        <specular>1.0 1.0 1.0</specular>
-        <direction>1 0 0</direction>
-        <intensity>0.5</intensity>
-        <spot>
-          <inner_angle>1.0</inner_angle>
-          <outer_angle>2.0</outer_angle>
-          <falloff>0.4</falloff>
-        </spot>
-        <attenuation>
-          <range>20.0</range>
-          <constant>1.0</constant>
-          <linear>1.0</linear>
-          <quadratic>1.0</quadratic>
-        </attenuation>
-      </light>
-    </gazebo>
-  </xacro:macro> -->
 </robot>

File: husarion_ugv_description/urdf/lynx.urdf.xacro (robot description, xacro)
@@ -22,5 +22,5 @@
   <xacro:arg name="components_config_path" default="$(find husarion_ugv_description)/config/components.yaml" />
   <xacro:property name="components_config_path_property" value="$(arg components_config_path)" />
-  <xacro:unless value="${components_config_path_property == 'None'}">
+  <!-- <xacro:unless value="${components_config_path_property == 'None'}">
     <xacro:include filename="$(find husarion_components_description)/urdf/components.urdf.xacro"
       ns="husarion_components" />
@@ -30,4 +30,4 @@
       use_sim="$(arg use_sim)"
     />
-  </xacro:unless>
+  </xacro:unless> -->
 </robot>

File: husarion_ugv_description/urdf/lynx/lynx_macro.urdf.xacro (robot description, xacro)
@@ -6,5 +6,5 @@
             controller_config_file
             battery_config_file
-            use_sim:=false
+            use_sim:=true
             imu_xyz:='0.052 0.073 -0.006'
             imu_rpy:='0.0 0.0 -1.57'
@@ -50,35 +50,5 @@
     <ros2_control name="${ns}lynx_system" type="system">
       <hardware>
-        <xacro:if value="${use_sim}">
-          <plugin>husarion_ugv_gazebo/EStopSystem</plugin>
-          <param name="e_stop_initial_state">false</param>
-        </xacro:if>
-        <xacro:unless value="${use_sim}">
-          <plugin>husarion_ugv_hardware_interfaces/LynxSystem</plugin>
-          <param name="encoder_resolution">1600</param>
-          <param name="gear_ratio">30.08</param>
-          <param name="gearbox_efficiency">0.75</param>
-          <!-- Same as set in the Roboteq driver (TNM parameter) -->
-          <param name="motor_torque_constant">0.11</param>
-          <!-- Max RPM speed set in the Roboteq driver (MXRPM parameter) -->
-          <param name="max_rpm_motor_speed">3600.0</param>
-          <param name="can_interface_name">robot_can</param>
-          <param name="master_can_id">3</param>
-          <param name="driver_can_id">1</param>
-          <param name="sdo_operation_timeout_ms">100</param>
-          <!-- Depends on frequency of the controller, more critical motors state are sent with
-            higher frequency, other parameters are sent with lower, here allowed time is set
-            to be expected period +50% margin -->
-          <param name="pdo_motor_states_timeout_ms">15</param>
-          <param name="pdo_driver_state_timeout_ms">75</param>
-          <!-- It will be rounded to the closest value taking into account current controller frequency -->
-          <param name="driver_states_update_frequency">20.0</param>
-          <param name="max_roboteq_initialization_attempts">5</param>
-          <param name="max_roboteq_activation_attempts">5</param>
-          <!-- TODO after all tests update parameters, these ones are quite high for the worst case scenario -->
-          <param name="max_write_pdo_cmds_errors_count">2</param>
-          <param name="max_read_pdo_motor_states_errors_count">2</param>
-          <param name="max_read_pdo_driver_state_errors_count">2</param>
-        </xacro:unless>
+        <plugin>gz_ros2_control/GazeboSimSystem</plugin>
       </hardware>
       <joint name="fl_wheel_joint">
@@ -161,6 +131,4 @@
       <xacro:gazebo.imu reference_frame="imu_link" namespace="${namespace}" />
       <!-- TODO Add lights visualization -->
-      <!-- <xacro:gazebo.light reference_frame="lights_channel_1_link" name="lights_channel_1" topic="lights/channel_1_frame" namespace="${namespace}" /> -->
-      <!-- <xacro:gazebo.light reference_frame="lights_channel_2_link" name="lights_channel_2" topic="lights/channel_2_frame" namespace="${namespace}" /> -->
     </xacro:if>
   </xacro:macro>

File: husarion_ugv_description/urdf/panther/panther_macro.urdf.xacro (robot description, xacro)
@@ -50,36 +50,5 @@
     <ros2_control name="${ns}panther_system" type="system">
       <hardware>
-        <xacro:if value="${use_sim}">
-          <plugin>husarion_ugv_gazebo/EStopSystem</plugin>
-          <param name="e_stop_initial_state">false</param>
-        </xacro:if>
-        <xacro:unless value="${use_sim}">
-          <plugin>husarion_ugv_hardware_interfaces/PantherSystem</plugin>
-          <param name="encoder_resolution">1600</param>
-          <param name="gear_ratio">30.08</param>
-          <param name="gearbox_efficiency">0.75</param>
-          <!-- Same as set in the Roboteq driver (TNM parameter) -->
-          <param name="motor_torque_constant">0.11</param>
-          <!-- Max RPM speed set in the Roboteq driver (MXRPM parameter) -->
-          <param name="max_rpm_motor_speed">3600.0</param>
-          <param name="can_interface_name">robot_can</param>
-          <param name="master_can_id">3</param>
-          <param name="front_driver_can_id">1</param>
-          <param name="rear_driver_can_id">2</param>
-          <param name="sdo_operation_timeout_ms">100</param>
-          <!-- Depends on frequency of the controller, more critical motors state are sent with
-            higher frequency, other parameters are sent with lower, here allowed time is set
-            to be expected period +50% margin -->
-          <param name="pdo_motor_states_timeout_ms">15</param>
-          <param name="pdo_driver_state_timeout_ms">75</param>
-          <!-- It will be rounded to the closest value taking into account current controller frequency -->
-          <param name="driver_states_update_frequency">20.0</param>
-          <param name="max_roboteq_initialization_attempts">5</param>
-          <param name="max_roboteq_activation_attempts">5</param>
-          <!-- TODO after all tests update parameters, these ones are quite high for the worst case scenario -->
-          <param name="max_write_pdo_cmds_errors_count">2</param>
-          <param name="max_read_pdo_motor_states_errors_count">2</param>
-          <param name="max_read_pdo_driver_state_errors_count">2</param>
-        </xacro:unless>
+        <plugin>gz_ros2_control/GazeboSimSystem</plugin>
       </hardware>
       <joint name="fl_wheel_joint">
